Commit message: Added camera functionality to assistive workspace Now you can view the camera feed in RViz and Gazebo. This will allow to have simulations with a camera feed for testing in simulation To do this we needed to create a world file for Gazebo instead of an empty world. Also added a separate camera xacro file for more modularity.

File: src/assistive_workspace_sim/urdf/workspace.urdf.xacro (robot description, xacro)
@@ -1,4 +1,5 @@
 <?xml version="1.0"?>
 <robot name="assistive_workspace" xmlns:xacro="http://ros.org/wiki/xacro">
+  <xacro:include filename="camera.xacro" />
   <link name="world"/>
   <link name="table_link">
@@ -50,19 +51,4 @@
     <origin xyz="0.25 0 0.8005" rpy="0 0 0"/>
   </joint>
-  <link name="camera_link">
-    <inertial>
-      <mass value="0.2"/>
-      <origin xyz="0 0 0" rpy="0 0 0"/>
-      <inertia ixx="0.001" ixy="0.0" ixz="0.0" iyy="0.001" iyz="0.0" izz="0.001"/>
-    </inertial>
-    <visual>
-      <geometry>
-        <box size="0.05 0.05 0.05"/>
-      </geometry>
-      <material name="black">
-        <color rgba="0 0 0 1"/>
-      </material>
-    </visual>
-  </link>
   <joint name="table_to_camera" type="fixed">
     <parent link="table_link"/>
@@ -70,24 +56,4 @@
     <origin xyz="0.25 0 1.3" rpy="0 1.5708 0"/>
   </joint>
-  <gazebo reference="camera_link">
-    <sensor name="vision_camera" type="camera">
-      <camera>
-        <horizontal_fov>1.047</horizontal_fov>
-        <image>
-          <width>640</width>
-          <height>480</height>
-          <format>R8G8B8</format>
-        </image>
-        <clip>
-          <near>0.01</near>
-          <far>2.0</far>
-        </clip>
-      </camera>
-      <always_on>1</always_on>
-      <update_rate>30</update_rate>
-      <visualize>true</visualize>
-      <topic>camera/image_raw</topic>
-    </sensor>
-  </gazebo>
   <gazebo reference="table_link">
     <material>
@@ -102,9 +68,3 @@
     </material>
   </gazebo>
-  <gazebo reference="camera_link">
-    <material>
-      <ambient>0.1 0.1 0.1 1.0</ambient>
-      <diffuse>0.1 0.1 0.1 1.0</diffuse>
-    </material>
-  </gazebo>
 </robot>
