Commit message: Custom moveit2 config package for 280pi gripper

File: src/mycobot_ros2/mycobot_description/urdf/mycobot_280_pi/mycobot_280_pi_adaptive_gripper.urdf (robot description, URDF)
Before this commit: robot firefighter, 15 links, 14 joints
Links:
- link g_base: mass 0.1 -> None; geometry collision cylinder length=0.05 radius=0.035; visual mesh filename=package://mycobot_description/urdf/mycobot_280_pi/G_base.dae
- link gripper_base: mass 0.1 -> None; geometry collision box size=0.04 0.04 0.03; visual mesh filename=package://mycobot_description/urdf/adaptive_gripper/gripper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
- link gripper_left1: mass 0.1 -> None; geometry collision box size=0.01 0.03 0.01; visual mesh filename=package://mycobot_description/urdf/adaptive_gripper/gripper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
- link gripper_left2: mass 0.1 -> None; geometry collision box size=0.01 0.03 0.01; visual mesh filename=package://mycobot_description/urdf/adaptive_gripper/gripper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
- link gripper_left3: mass 0.1 -> None; geometry collision box size=0.01 0.03 0.01; visual mesh filename=package://mycobot_description/urdf/adaptive_gripper/gripper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
- link gripper_right1: mass 0.1 -> None; geometry collision box size=0.01 0.03 0.01; visual mesh filename=package://mycobot_description/urdf/adaptive_gripper/gripper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
- link gripper_right2: mass 0.1 -> None; geometry collision box size=0.01 0.03 0.01; visual mesh filename=package://mycobot_description/urdf/adaptive_gripper/gripper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
- link gripper_right3: mass 0.1 -> None; geometry collision box size=0.01 0.03 0.01; visual mesh filename=package://mycobot_description/urdf/adaptive_gripper/gripper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
- link joint1: mass 0.1 -> None; geometry collision cylinder length=0.06 radius=0.03; visual mesh filename=package://mycobot_description/urdf/mycobot_280_pi/joint1_pi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
- link joint2: mass 0.1 -> None; geometry collision cylinder length=0.11 radius=0.025; visual mesh filename=package://mycobot_description/urdf/mycobot_280_pi/joint2.dae
- link joint3: mass 0.1 -> None; geometry collision cylinder length=0.11 radius=0.025; visual mesh filename=package://mycobot_description/urdf/mycobot_280_pi/joint3.dae
- link joint4: mass 0.1 -> None; geometry collision cylinder length=0.07 radius=0.025; visual mesh filename=package://mycobot_description/urdf/mycobot_280_pi/joint4.dae
- link joint5: mass 0.1 -> None; geometry collision cylinder length=0.07 radius=0.025; visual mesh filename=package://mycobot_description/urdf/mycobot_280_pi/joint5.dae
- link joint6: mass 0.1 -> None; geometry collision cylinder length=0.04 radius=0.02; visual mesh filename=package://mycobot_description/urdf/mycobot_280_pi/joint6.dae
- link joint6_flange: mass 0.1 -> None; geometry collision cylinder length=0.01 radius=0.015; visual mesh filename=package://mycobot_description/urdf/mycobot_280_pi/joint7.dae
Joints:
- joint g_base_to_joint1: axis 0 0 0 -> 0 0 1
- joint gripper_base_to_gripper_left2: limit lower=-0.8 upper=0.5 effort=1000.0 velocity=0 -> lower=-3.14 upper=3.14 effort=1000.0 velocity=0
- joint gripper_base_to_gripper_right2: limit lower=-0.5 upper=0.8 effort=1000.0 velocity=0 -> lower=-3.14 upper=3.14 effort=1000.0 velocity=0
- joint gripper_base_to_gripper_right3: limit lower=-0.15 upper=0.7 effort=1000.0 velocity=0 -> lower=-3.14 upper=3.14 effort=1000.0 velocity=0
- joint gripper_controller: limit lower=-0.74 upper=0.15 effort=1000.0 velocity=0 -> lower=-3.14 upper=3.14 effort=1000.0 velocity=0
- joint gripper_left3_to_gripper_left1: limit lower=-0.5 upper=0.5 effort=1000.0 velocity=0 -> lower=-3.14 upper=3.14 effort=1000.0 velocity=0
- joint gripper_right3_to_gripper_right1: limit lower=-0.5 upper=0.5 effort=1000.0 velocity=0 -> lower=-3.14 upper=3.14 effort=1000.0 velocity=0

Commit message: Updated urdf visualizualizing joints 1&5 in gazebo Before needed shapes in place of joints for gazebo Changed dae files into stl files

File: src/mycobot_ros2/mycobot_description/urdf/mycobot_280_pi/mycobot_280_pi_adaptive_gripper.urdf (robot description, URDF)
Before this commit: robot firefighter, 15 links, 14 joints
Links:
- link g_base: mass None -> 0.1
- link gripper_base: mass None -> 0.1
- link gripper_left1: mass None -> 0.1
- link gripper_left2: mass None -> 0.1
- link gripper_left3: mass None -> 0.1
- link gripper_right1: mass None -> 0.1
- link gripper_right2: mass None -> 0.1
- link gripper_right3: mass None -> 0.1
- link joint1: mass None -> 0.1
- link joint2: mass None -> 0.1
- link joint3: mass None -> 0.1
- link joint4: mass None -> 0.1
- link joint5: mass None -> 0.1; geometry collision cylinder length=0.07 radius=0.025; visual mesh filename=package://mycobot_description/urdf/mycobot_280_pi/joint5.stl
- link joint6: mass None -> 0.1
- link joint6_flange: mass None -> 0.1
